Commit message: feat: added a new dimension z for more possibilities such that there is new angles that are formed and more configurations possible for the robotic arm

File: install/my_robot/share/my_robot/urdf/robot_arm.urdf (robot description, URDF)
Before this commit: robot robot_arm_horizontal, 7 links, 6 joints
Links:
- removed link shoulder
- added link base_link, mass 1.0; visual cylinder length=0.05 radius=0.07
Joints:
- removed joint claw_base_joint
- removed joint elbow_joint
- removed joint shoulder_joint
- removed joint wrist_joint
- added joint base_yaw: type continuous, parent world, child base_link, origin xyz=0 0 0 rpy=0 0 0, axis 0 0 1, limit effort=10 velocity=1.0
- added joint elbow_pitch: type continuous, parent upper_arm, child forearm, origin xyz=0.4 0 0 rpy=0 0 0, axis 0 1 0, limit effort=5 velocity=1.0
- added joint shoulder_pitch: type continuous, parent base_link, child upper_arm, origin xyz=0.05 0 0 rpy=0 0 0, axis 0 1 0, limit effort=10 velocity=1.0
- added joint wrist_pitch: type continuous, parent forearm, child claw_base, origin xyz=0.3 0 0 rpy=0 0 0, axis 0 1 0, limit effort=5 velocity=1.0
